Commit message: fixed file names

File: redcat_bringup/urdf/robot_core.xacro (robot description, xacro)
@@ -16,5 +16,5 @@
             <origin xyz="0 0 0" rpy="0 0 0"/>
             <geometry>
-                <mesh filename="package://redcat_bringup/meshes/base_link.STL" size="${scale_factor}"/>
+                <mesh filename="package://redcat_bringup/meshes/car_body.STL" size="${scale_factor}"/>
             </geometry>
             <material name="grey"/>
@@ -23,5 +23,5 @@
             <origin xyz="0 0 0" rpy="0 0 0"/>
             <geometry>
-                <mesh filename="package://redcat_bringup/meshes/collision/base_link.STL" size="${scale_factor}"/>
+                <mesh filename="package://redcat_bringup/meshes/collision/car_body.STL" size="${scale_factor}"/>
             </geometry>
         </collision>

File: redcat_bringup/urdf/sensors.xacro (robot description, xacro)
@@ -4,9 +4,9 @@
     <!-- ************************************ Unitree L2  ***************************************** -->
     <!-- ****************************************************************************************** -->
-    <link name="unitree_l2">
+    <link name="unitree_L2">
         <visual>
             <origin xyz="0 0 0" rpy="0 0 0"/>
             <geometry>
-                <mesh filename="package://redcat_bringup/meshes/unitree_l2.STL" size="${scale_factor}"/>
+                <mesh filename="package://redcat_bringup/meshes/L2_lidar.STL" size="${scale_factor}"/>
             </geometry>
             <material name="black"/>
@@ -15,11 +15,11 @@
             <origin xyz="0 0 0" rpy="0 0 0"/>
             <geometry>
-                <mesh filename="package://redcat_bringup/meshes/unitree_l2.STL" size="${scale_factor}"/>
+                <mesh filename="package://redcat_bringup/meshes/L2_lidar.STL" size="${scale_factor}"/>
             </geometry>
         </collision>
     </link>
-    <joint name="unitree_l2_joint" type="fixed">
+    <joint name="unitree_L2_joint" type="fixed">
         <parent link="base_link"/>
-        <child link="unitree_l2"/>
+        <child link="unitree_L2"/>
         <origin xyz="0 0.1026 0.0915" rpy="0 0 0"/>
     </joint>

Commit message: ros2_control configuration

File: redcat_bringup/urdf/robot_core.xacro (robot description, xacro)
@@ -16,5 +16,5 @@
             <origin xyz="0 0 0" rpy="0 0 0"/>
             <geometry>
-                <mesh filename="package://redcat_bringup/meshes/car_body.STL" size="${scale_factor}"/>
+                <mesh filename="package://redcat_bringup/meshes/car_body.stl" scale="${scale_factor}"/>
             </geometry>
             <material name="grey"/>
@@ -23,5 +23,5 @@
             <origin xyz="0 0 0" rpy="0 0 0"/>
             <geometry>
-                <mesh filename="package://redcat_bringup/meshes/collision/car_body.STL" size="${scale_factor}"/>
+                <mesh filename="package://redcat_bringup/meshes/collision/car_body.stl" scale="${scale_factor}"/>
             </geometry>
         </collision>
@@ -33,5 +33,25 @@
     </joint>
     <!-- ****************************************************************************************** -->
-    <!-- ********************************* Front Left Wheel  ************************************** -->
+    <!-- ************************************* Steering  ****************************************** -->
+    <!-- ****************************************************************************************** -->
+    <link name="fl_steering_link"/>
+    <link name="fr_steering_link"/>
+    <joint name="steering_joint" type="revolute">
+        <parent link="base_link"/>
+        <child link="fl_steering_link"/>
+        <origin xyz="-0.1125 0.1405 0.0121" rpy="0 0 0"/>
+        <axis xyz="0 0 1"/>
+        <limit lower="${-pi/6}" upper="${pi/6}" effort="1" velocity="10"/>
+    </joint>
+    <joint name="steering_mimic_joint" type="revolute">
+        <parent link="base_link"/>
+        <child link="fr_steering_link"/>
+        <origin xyz="0.1125 0.1405 0.0121" rpy="0 0 0"/>
+        <axis xyz="0 0 1"/>
+        <limit lower="${-pi/6}" upper="${pi/6}" effort="1" velocity="10"/>
+        <mimic joint="steering_joint" multiplier="1" offset="0"/>
+    </joint>
+    <!-- ****************************************************************************************** -->
+    <!-- ********************************* Front Left Drive  ************************************** -->
     <!-- ****************************************************************************************** -->
     <link name="fl_wheel">
@@ -39,5 +59,5 @@
             <origin xyz="0 0 0" rpy="0 0 0"/>
             <geometry>
-                <mesh filename="package://redcat_bringup/meshes/wheel.STL" size="${scale_factor}"/>
+                <mesh filename="package://redcat_bringup/meshes/wheel.stl" scale="${scale_factor}"/>
             </geometry>
             <material name="black"/>
@@ -46,16 +66,16 @@
             <origin xyz="0 0 0" rpy="0 0 0"/>
             <geometry>
-                <mesh filename="package://redcat_bringup/meshes/collision/wheel.STL" size="${scale_factor}"/>
+                <mesh filename="package://redcat_bringup/meshes/collision/wheel.stl" scale="${scale_factor}"/>
             </geometry>
         </collision>
     </link>
-    <joint name="fl_wheel_joint" type="continuous">
-        <parent link="base_link"/>
+    <joint name="drive_joint" type="continuous">
+        <parent link="fl_steering_link"/>
         <child link="fl_wheel"/>
-        <origin xyz="-0.1125 0.1405 0.0121" rpy="0 -${pi/2} 0"/>
+        <origin xyz="0 0 0" rpy="0 -${pi/2} 0"/>
         <axis xyz="0 0 1"/>
     </joint>
     <!-- ****************************************************************************************** -->
-    <!-- ********************************* Front Right Wheel  ************************************* -->
+    <!-- ********************************* Front Right Drive  ************************************* -->
     <!-- ****************************************************************************************** -->
     <link name="fr_wheel">
@@ -63,5 +83,5 @@
             <origin xyz="0 0 0" rpy="0 0 0"/>
             <geometry>
-                <mesh filename="package://redcat_bringup/meshes/wheel.STL" size="${scale_factor}"/>
+                <mesh filename="package://redcat_bringup/meshes/wheel.stl" scale="${scale_factor}"/>
             </geometry>
             <material name="black"/>
@@ -70,16 +90,17 @@
             <origin xyz="0 0 0" rpy="0 0 0"/>
             <geometry>
-                <mesh filename="package://redcat_bringup/meshes/collision/wheel.STL" size="${scale_factor}"/>
+                <mesh filename="package://redcat_bringup/meshes/collision/wheel.stl" scale="${scale_factor}"/>
             </geometry>
         </collision>
     </link>
     <joint name="fr_wheel_joint" type="continuous">
-        <parent link="base_link"/>
+        <parent link="fr_steering_link"/>
         <child link="fr_wheel"/>
-        <origin xyz="0.1125 0.1405 0.0121" rpy="0 ${pi/2} 0"/>
+        <origin xyz="0 0 0" rpy="0 ${pi/2} 0"/>
         <axis xyz="0 0 1"/>
+        <mimic joint="drive_joint" multiplier="-1" offset="0"/>
     </joint>
     <!-- ****************************************************************************************** -->
-    <!-- ********************************* Rear Left Wheel  *************************************** -->
+    <!-- ********************************* Rear Left Drive  *************************************** -->
     <!-- ****************************************************************************************** -->
     <link name="rl_wheel">
@@ -87,5 +108,5 @@
             <origin xyz="0 0 0" rpy="0 0 0"/>
             <geometry>
-                <mesh filename="package://redcat_bringup/meshes/wheel.STL" size="${scale_factor}"/>
+                <mesh filename="package://redcat_bringup/meshes/wheel.stl" scale="${scale_factor}"/>
             </geometry>
             <material name="black"/>
@@ -94,5 +115,5 @@
             <origin xyz="0 0 0" rpy="0 0 0"/>
             <geometry>
-                <mesh filename="package://redcat_bringup/meshes/collision/wheel.STL" size="${scale_factor}"/>
+                <mesh filename="package://redcat_bringup/meshes/collision/wheel.stl" scale="${scale_factor}"/>
             </geometry>
         </collision>
@@ -103,7 +124,8 @@
         <origin xyz="-0.1125 -0.1405 0.0121" rpy="0 -${pi/2} 0"/>
         <axis xyz="0 0 1"/>
+        <mimic joint="drive_joint" multiplier="1" offset="0"/>
     </joint>
     <!-- ****************************************************************************************** -->
-    <!-- ********************************* Rear Right Wheel  *************************************** -->
+    <!-- ********************************* Rear Right Drive  *************************************** -->
     <!-- ****************************************************************************************** -->
     <link name="rr_wheel">
@@ -111,5 +133,5 @@
             <origin xyz="0 0 0" rpy="0 0 0"/>
             <geometry>
-                <mesh filename="package://redcat_bringup/meshes/wheel.STL" size="${scale_factor}"/>
+                <mesh filename="package://redcat_bringup/meshes/wheel.stl" scale="${scale_factor}"/>
             </geometry>
             <material name="black"/>
@@ -118,5 +140,5 @@
             <origin xyz="0 0 0" rpy="0 0 0"/>
             <geometry>
-                <mesh filename="package://redcat_bringup/meshes/collision/wheel.STL" size="${scale_factor}"/>
+                <mesh filename="package://redcat_bringup/meshes/collision/wheel.stl" scale="${scale_factor}"/>
             </geometry>
         </collision>
@@ -127,4 +149,5 @@
         <origin xyz="0.1125 -0.1405 0.0121" rpy="0 ${pi/2} 0"/>
         <axis xyz="0 0 1"/>
+        <mimic joint="drive_joint" multiplier="-1" offset="0"/>
     </joint>
 </robot>

File: redcat_bringup/urdf/ros2_control.xacro (robot description, xacro)
@@ -17,11 +17,11 @@
                 </hardware>
             </xacro:if>
-            <joint name="rl_wheel_joint">
+            <joint name="drive_joint">
                 <command_interface name="velocity"/>
                 <state_interface name="velocity"/>
             </joint>
-            <joint name="fr_wheel_joint">
-                <command_interface name="velocity"/>
-                <state_interface name="velocity"/>
+            <joint name="steering_joint">
+                <command_interface name="position"/>
+                <state_interface name="position"/>
             </joint>
         </ros2_control>

File: redcat_bringup/urdf/sensors.xacro (robot description, xacro)
@@ -8,5 +8,5 @@
             <origin xyz="0 0 0" rpy="0 0 0"/>
             <geometry>
-                <mesh filename="package://redcat_bringup/meshes/L2_lidar.STL" size="${scale_factor}"/>
+                <mesh filename="package://redcat_bringup/meshes/L2_lidar.stl" scale="${scale_factor}"/>
             </geometry>
             <material name="black"/>
@@ -15,5 +15,5 @@
             <origin xyz="0 0 0" rpy="0 0 0"/>
             <geometry>
-                <mesh filename="package://redcat_bringup/meshes/L2_lidar.STL" size="${scale_factor}"/>
+                <mesh filename="package://redcat_bringup/meshes/L2_lidar.stl" scale="${scale_factor}"/>
             </geometry>
         </collision>

Commit message: debugging world frame error

File: redcat_bringup/urdf/robot_core.xacro (robot description, xacro)
@@ -11,5 +11,4 @@
     <!-- ***************************************** Base ******************************************* -->
     <!-- ****************************************************************************************** -->
-    <link name="world" />
     <link name="base_link">
         <visual>
@@ -27,9 +26,4 @@
         </collision>
     </link>
-    <joint name="base_joint" type="fixed">
-        <parent link="world"/>
-        <child link="base_link"/>
-        <origin xyz="0 0 0" rpy="0 0 0"/>
-    </joint>
     <!-- ****************************************************************************************** -->
     <!-- ************************************* Steering  ****************************************** -->
