Commit message: slam_toolbox config

File: redcat/urdf/robot_core.xacro (robot description, xacro)
@@ -11,5 +11,12 @@
     <!-- ***************************************** Base ******************************************* -->
     <!-- ****************************************************************************************** -->
-    <link name="base_link">
+    <link name="base_link"/>
+    <link name="base_footprint"/>
+    <joint name="base_link_joint" type="fixed">
+        <parent link="base_link"/>
+        <child link="base_footprint"/>
+        <origin xyz="0 0 0" rpy="0 0 0"/>
+    </joint>
+    <link name="chassis">
         <visual>
             <origin xyz="0 0 0" rpy="0 0 0"/>
@@ -26,4 +33,9 @@
         </collision>
     </link>
+    <joint name="chassis_joint" type="fixed">
+        <parent link="base_link"/>
+        <child link="chassis"/>
+        <origin xyz="0 0 0.0121" rpy="0 0 0"/>
+    </joint>
     <!-- ****************************************************************************************** -->
     <!-- ************************************* Steering  ****************************************** -->
@@ -32,5 +44,5 @@
     <link name="fr_steering_link"/>
     <joint name="steering_joint" type="revolute">
-        <parent link="base_link"/>
+        <parent link="chassis"/>
         <child link="fl_steering_link"/>
         <origin xyz="-0.1125 0.1405 0.0121" rpy="0 0 0"/>
@@ -39,5 +51,5 @@
     </joint>
     <joint name="steering_mimic_joint" type="revolute">
-        <parent link="base_link"/>
+        <parent link="chassis"/>
         <child link="fr_steering_link"/>
         <origin xyz="0.1125 0.1405 0.0121" rpy="0 0 0"/>
@@ -114,5 +126,5 @@
     </link>
     <joint name="rl_wheel_joint" type="continuous">
-        <parent link="base_link"/>
+        <parent link="chassis"/>
         <child link="rl_wheel"/>
         <origin xyz="-0.1125 -0.1405 0.0121" rpy="0 -${pi/2} 0"/>
@@ -139,5 +151,5 @@
     </link>
     <joint name="rr_wheel_joint" type="continuous">
-        <parent link="base_link"/>
+        <parent link="chassis"/>
         <child link="rr_wheel"/>
         <origin xyz="0.1125 -0.1405 0.0121" rpy="0 ${pi/2} 0"/>

Commit message: controller tuning

File: redcat/urdf/robot_core.xacro (robot description, xacro)
@@ -18,4 +18,9 @@
         <origin xyz="0 0 0" rpy="0 0 0"/>
     </joint>
+    <joint name="chassis_joint" type="fixed">
+        <parent link="base_link"/>
+        <child link="chassis"/>
+        <origin xyz="0 0 0" rpy="0 0 0"/>
+    </joint>
     <link name="chassis">
         <visual>
@@ -33,9 +38,4 @@
         </collision>
     </link>
-    <joint name="chassis_joint" type="fixed">
-        <parent link="base_link"/>
-        <child link="chassis"/>
-        <origin xyz="0 0 0.0121" rpy="0 0 0"/>
-    </joint>
     <!-- ****************************************************************************************** -->
     <!-- ************************************* Steering  ****************************************** -->

File: redcat/urdf/ros2_control.xacro (robot description, xacro)
@@ -19,4 +19,6 @@
             <joint name="drive_joint">
                 <command_interface name="velocity"/>
+                    <param name="min">-10.0</param>
+                    <param name="max">10.0</param>
                 <state_interface name="position"/>
                 <state_interface name="velocity"/>
@@ -24,4 +26,6 @@
             <joint name="steering_joint">
                 <command_interface name="position"/>
+                <param name="min">${-pi/6}</param>
+                <param name="max">${pi/6}</param>
                 <state_interface name="position"/>
             </joint>

File: redcat/urdf/sensors.xacro (robot description, xacro)
@@ -20,5 +20,5 @@
     </link>
     <joint name="unitree_L2_joint" type="fixed">
-        <parent link="base_link"/>
+        <parent link="chassis"/>
         <child link="unitree_L2"/>
         <origin xyz="0 0.1026 0.0915" rpy="0 0 0"/>
