Commit message: isaacsim RTX lidar integration

File: redcat/urdf/robot.urdf.xacro (robot description, xacro)
@@ -2,5 +2,5 @@
 <robot xmlns:xacro="http://www.ros.org/wiki/xacro"  name="redcat_car">
     <xacro:arg name="HW_mode" default="mock"/>
-    <xacro:include filename="robot_core.xacro"/>
+    <xacro:include filename="robot_core_diff.xacro"/>
     <xacro:include filename="sensors.xacro"/>
     <xacro:include filename="ros2_control.xacro"/>

File: redcat/urdf/ros2_control.xacro (robot description, xacro)
@@ -17,5 +17,5 @@
                 </hardware>
             </xacro:if>
-            <joint name="drive_joint">
+            <joint name="fl_wheel_joint">
                 <command_interface name="velocity"/>
                     <param name="min">-10.0</param>
@@ -24,9 +24,24 @@
                 <state_interface name="velocity"/>
             </joint>
-            <joint name="steering_joint">
-                <command_interface name="position"/>
-                <param name="min">${-pi/6}</param>
-                <param name="max">${pi/6}</param>
+            <joint name="fr_wheel_joint">
+                <command_interface name="velocity"/>
+                    <param name="min">-10.0</param>
+                    <param name="max">10.0</param>
                 <state_interface name="position"/>
+                <state_interface name="velocity"/>
+            </joint>
+            <joint name="rl_wheel_joint">
+                <command_interface name="velocity"/>
+                    <param name="min">-10.0</param>
+                    <param name="max">10.0</param>
+                <state_interface name="position"/>
+                <state_interface name="velocity"/>
+            </joint>
+            <joint name="rr_wheel_joint">
+                <command_interface name="velocity"/>
+                    <param name="min">-10.0</param>
+                    <param name="max">10.0</param>
+                <state_interface name="position"/>
+                <state_interface name="velocity"/>
             </joint>
         </ros2_control>
